File: SchematicWeatherIC.sch (EAGLE design)
At the start: 32 parts

Commit message: use smaller resistors and autoroute
Parts:
- R1, R2: device rcl:R-EU_0204/7 -> rcl:R-US_VMTA55
- R3, R4, R5, R6, R7, R8, R9: device rcl:R-US_VMTB60 -> rcl:R-US_VMTA55
Connections:
- net GND: now also R6.1, R7.1; no longer R6.2, R7.2
- net N$12: now also R6.2; no longer R6.1
- net N$13: now also R7.2; no longer R7.1
- net N$2: now also R8.2; no longer R9.1
- net N$3: now also R9.1; no longer R8.2
- net N$6: now also R8.1; no longer R9.2
- net VDD: now also R9.2; no longer R8.1
Other:
- moved on the sheet: R6, R7, R8, R9

Commit message: some wiring and routing updates in progress
Connections:
- new net N$20: ESP32.USB_D+/GPIO13, USBTOSERIAL.D+
- new net N$21: ESP32.USB_D-/GPIO12, USBTOSERIAL.D-
Changed lines of the file:
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@@
+</segment>
+</net>
+<net name="N$20" class="0">
+<segment>
+<pinref part="USBTOSERIAL" gate="G$1" pin="D+"/>
+<wire x1="137.16" y1="137.16" x2="121.92" y2="137.16" width="0.1524" layer="91"/>
+<wire x1="121.92" y1="137.16" x2="121.92" y2="106.68" width="0.1524" layer="91"/>
+<wire x1="121.92" y1="106.68" x2="246.38" y2="106.68" width="0.1524" layer="91"/>
+<wire x1="246.38" y1="106.68" x2="246.38" y2="78.74" width="0.1524" layer="91"/>
+<pinref part="ESP32" gate="G$1" pin="USB_D+/GPIO13"/>
+<wire x1="246.38" y1="78.74" x2="231.14" y2="78.74" width="0.1524" layer="91"/>
+</segment>
+</net>
+<net name="N$21" class="0">
+<segment>
+<pinref part="ESP32" gate="G$1" pin="USB_D-/GPIO12"/>
+<wire x1="231.14" y1="81.28" x2="248.92" y2="81.28" width="0.1524" layer="91"/>
+<wire x1="248.92" y1="81.28" x2="248.92" y2="109.22" width="0.1524" layer="91"/>
+<wire x1="248.92" y1="109.22" x2="134.62" y2="109.22" width="0.1524" layer="91"/>
+<pinref part="USBTOSERIAL" gate="G$1" pin="D-"/>
+<wire x1="134.62" y1="109.22" x2="134.62" y2="134.62" width="0.1524" layer="91"/>
+<wire x1="134.62" y1="134.62" x2="137.16" y2="134.62" width="0.1524" layer="91"/>
 </segment>
 </net>

Commit message: routed differential pair and i2c
Connections:
- net N$20 renamed D_P
- net N$21 renamed D_N
Changed lines of the file:
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@@
 <class number="0" name="default" width="0" drill="0">
+</class>
+<class number="1" name="differential_pair" width="0" drill="0">
 </class>
 </classes>
@@
 </segment>
 </net>
-<net name="N$20" class="0">
+<net name="D_P" class="1">
 <segment>
 <pinref part="USBTOSERIAL" gate="G$1" pin="D+"/>
@@
 </segment>
 </net>
-<net name="N$21" class="0">
+<net name="D_N" class="1">
 <segment>
 <pinref part="ESP32" gate="G$1" pin="USB_D-/GPIO12"/>
